File: eagle/pinoccio-wifi.brd (EAGLE design)
At the start: 25.4 x 55.4 mm, 23 parts, among them J1 AVR_SPI_PRG_6, J2 AVR_SPI_PRG_6, U1 GS1011MIPS, U2 M25PX16, U3 M25PX16, U4 TPS73533, U5 ATTINY13A

Commit message: Fix #1: typo for VUSB
Connections:
- net VBUS renamed VUSB
Changed lines of the file:
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@@
 <wire x1="20.788" y1="51.2972" x2="22.4988" y2="51.2972" width="0.2032" layer="1"/>
 </signal>
-<signal name="VBUS">
+<signal name="VUSB">
 <contactref element="JP-L" pad="P$1"/>
 </signal>

Commit message: Version 1.1 PCB update
- Connect D5 to Gainspan module GPIO28, for data-ready signal on SPI bus
- Connect ATTiny13A PB3 to Gainspan module reset pin, with 10k pull-up
Parts:
- added R7: 10k, Pinoccio:0402-RES
- moved C4 0.54 mm to (15.5, 26.4), turned to 90 degrees
Connections:
- new net WIFI-RESET: R7.2, U1.P$33, U5.2
- net D5: now also U1.P$2
- net WIFI-VCC: now also R7.1
Routing:
- net D5: track 0.00 -> 45.3 mm
- net WIFI-RESET: track 0.00 -> 38.4 mm, vias 0 -> 2
- net WIFI-VCC: track 33.7 -> 53.3 mm, vias 2 -> 4
- net GND: track 22.1 -> 8.77 mm, vias 18 -> 21
- net SCK: track 79.4 -> 82.4 mm
- net VBAT: track 29.0 -> 30.4 mm
- net MOSI: track 79.0 -> 80.4 mm
- net D6: track 49.0 -> 50.3 mm
- net VCC-AE: track 111.2 -> 112.3 mm
- net N$4: track 20.1 -> 21.1 mm
- net MISO: track 78.9 -> 79.9 mm
Other:
- board text added: "2014-03-10"
- board text added: "Pinoccio(tm) Wi-Fi Backpack v1.1"
- board text added: "wi-fi backpack v1.1"
- board text removed: "2013-08-15"
- board text removed: "Pinoccio(tm) Wi-Fi Backpack v1.0"
- board text removed: "wi-fi backpack v1.0"
