File: eagle/pinoccio-wifi.brd (EAGLE design)
At the start: 25.4 x 55.4 mm, 23 parts, among them J1 AVR_SPI_PRG_6, J2 AVR_SPI_PRG_6, U1 GS1011MIPS, U2 M25PX16, U3 M25PX16, U4 TPS73533, U5 ATTINY13A

Commit message: Add v1.1 changes
Other:
- board text added: "2014-03-29"
- board text added: "Pinoccio(tm) Wi-Fi Backpack v1.1"
- board text added: "wi-fi backpack v1.1"
- board text removed: "2013-08-15"
- board text removed: "Pinoccio(tm) Wi-Fi Backpack v1.0"
- board text removed: "wi-fi backpack v1.0"
Changed lines of the file:
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@@
 <text x="22.606" y="29.8958" size="1.016" layer="21" font="vector" ratio="15" rot="R180">SCL</text>
 <text x="-10.414" y="-6.604" size="1.27" layer="51" font="vector" ratio="15">Design by: Eric Jennings for Pinoccio</text>
-<text x="-10.3632" y="-4.8514" size="1.778" layer="51" font="vector" ratio="15">Pinoccio(tm) Wi-Fi Backpack v1.0</text>
+<text x="-10.3632" y="-4.8514" size="1.778" layer="51" font="vector" ratio="15">Pinoccio(tm) Wi-Fi Backpack v1.1</text>
 <wire x1="0" y1="8.128" x2="0" y2="63.5" width="0.2032" layer="20"/>
 <wire x1="0" y1="63.5" x2="25.4" y2="63.5" width="0.2032" layer="20"/>
@@
 <wire x1="0" y1="8.128" x2="25.4" y2="8.128" width="0.2032" layer="20"/>
 <circle x="12.7" y="29.845" radius="2.54" width="0.4064" layer="20"/>
-<text x="18.8976" y="61.6458" size="0.8128" layer="22" font="vector" ratio="15" rot="MR0">wi-fi backpack v1.0</text>
+<text x="18.8976" y="61.6458" size="0.8128" layer="22" font="vector" ratio="15" rot="MR0">wi-fi backpack v1.1</text>
 <text x="17.9832" y="60.2234" size="0.8128" layer="22" font="vector" ratio="15" rot="MR0">http://pinocc.io</text>
 <text x="14.986" y="41.4528" size="0.8128" layer="22" font="vector" ratio="15" rot="MR0">tiny13A</text>
 <text x="15.7734" y="49.7078" size="0.8128" layer="22" font="vector" ratio="15" rot="MR0">GS1011 SF</text>
-<text x="16.5608" y="58.6486" size="0.8128" layer="22" font="vector" ratio="15" rot="MR0">2013-08-15</text>
+<text x="16.5608" y="58.6486" size="0.8128" layer="22" font="vector" ratio="15" rot="MR0">2014-03-29</text>
 </plain>
 <attributes>

Commit message: Add data-ready trace to D5
Connections:
- net D5: now also U1.P$2
Routing:
- net D5: track 0.00 -> 45.1 mm
- net GND: vias 18 -> 20
Changed lines of the file:
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@@
 <via x="16.9672" y="42.799" extent="1-16" drill="0.4064"/>
 <via x="16.9672" y="45.339" extent="1-16" drill="0.4064"/>
+<via x="3.7338" y="42.6974" extent="1-16" drill="0.4064"/>
+<via x="3.7084" y="40.5384" extent="1-16" drill="0.4064"/>
 </signal>
 <signal name="WIFI-VCC" class="1">
@@
 <signal name="D5">
 <contactref element="JP-L" pad="P$13"/>
+<contactref element="U1" pad="P$2"/>
+<wire x1="1.651" y1="15.37" x2="0.6604" y2="16.3606" width="0.2032" layer="1"/>
+<wire x1="0.6604" y1="16.3606" x2="0.6604" y2="57.2008" width="0.2032" layer="1"/>
+<wire x1="0.6604" y1="57.2008" x2="1.7568" y2="58.2972" width="0.2032" layer="1"/>
+<wire x1="1.7568" y1="58.2972" x2="3.0988" y2="58.2972" width="0.2032" layer="1"/>
 </signal>
 <signal name="D6">
